File: HMKB70/HMKB70_Nicenano_LED.kicad_pcb (KiCad board)
At the start: 2 copper layers, 169 parts, among them U1 Nice_Nano_V2

Commit message: 1u footprint fix and misc other
Fixed 1u MX switch footprint, changed LED line to an ugly magenta, fixed LED circuit with current drain.
Parts:
- moved D3_F2 37.1 mm to (72.2, 24.1)
- moved D2_F1 14.6 mm to (52.9, 24.2)
- moved S2_F1 6.63 mm to (44.8, 21.6)
- moved S3_F2 6.63 mm to (63.9, 21.6)
- moved D28_PROG3 3.68 mm to (340.6, 46.8)
- moved D40 3.68 mm to (167.4, 126.0)
- moved D44_PROG4 3.68 mm to (341.0, 67.2)
- moved S20_6 3.68 mm to (139.1, 48.8)
- moved S21_7 3.68 mm to (158.1, 48.8)
- moved S22_8 3.68 mm to (177.1, 48.7)
- moved S23_9 3.68 mm to (196.2, 48.7)
- moved S24_0 3.68 mm to (215.3, 48.7)
- moved S26_=1 3.68 mm to (253.2, 48.8)
- moved S33 3.68 mm to (134.6, 90.4)
- moved S34_T1 3.68 mm to (134.2, 70.0)
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